File: KiCAD/Switch3V/Switch3Vx.kicad_pcb (KiCad board)
At the start: 2 copper layers, 31.8 x 17.8 mm, 15 parts, among them J1 ESP8266-12F, J2 1-Wite, J3 Relay, Q1 BC547, Q2 BSS138, SW1 SW_Push, U1 LM1117-3.3

Commit message: porawiono pliki kiCAD
Routing:
- net GND: track 38.0 -> 49.9 mm
- net Net-(J1-Pad4): track 38.1 -> 36.3 mm
- net Net-(D1-Pad2): track 30.1 -> 30.2 mm, vias 0 -> 2
